File: HW/wcube-fan-pcb..kicad_pcb (KiCad board)
At the start: 2 copper layers, 60 x 18 mm, 40 parts, among them J1 HOT_END, J2 ON_~OFF, J3 POWER, M1 Fan, M2 Fan, M3 Fan, M4 Fan, Q1 BC817, Q2 BC817, Q3 BC817, Q4 BC807, Q5 BC807, Q6 BC807, U1 ATTINY13A-SSU, U2 L78L05_SO8

Commit message: Swapped ADC pins
Connections:
- C1 pad 1: /ADC_HEAD -> /ADC_BOX
- C2 pad 1: /ADC_BOX -> /ADC_HEAD
- RV1 pad 2: /ADC_HEAD -> /ADC_BOX
- RV2 pad 2: /ADC_BOX -> /ADC_HEAD
- U1 pad 2: /ADC_HEAD -> /ADC_BOX
- U1 pad 3: /ADC_BOX -> /ADC_HEAD
Routing:
- net /ADC_HEAD: track 17.3 -> 10.4 mm
- net /ADC_BOX: track 10.4 -> 17.3 mm
